Commit message: 0320

File: Smartcart_ROS/kobuki/kobuki_description/urdf/kobuki.urdf.xacro (robot description, xacro)
@@ -222,5 +222,5 @@
       <link name="base_scan">
         <visual>
-          <origin xyz="0 0 0.0" rpy="0 0 0"/>
+          <origin xyz="0 0 0.0" rpy="0 0 3.14159"/>
           <geometry>
             <mesh filename="package://kobuki_description/meshes/sensors/lds.stl" scale="0.001 0.001 0.001"/>
@@ -229,5 +229,5 @@
         </visual>
         <collision>
-          <origin xyz="0.015 0 -0.0065" rpy="0 0 0"/>
+          <origin xyz="0.015 0 -0.0065" rpy="0 0 3.14159"/>
           <geometry>
             <cylinder length="0.0315" radius="0.045"/>

File: Smartcart_ROS/kobuki/kobuki_description/urdf/kobuki_gazebo.urdf.xacro (robot description, xacro)
@@ -188,8 +188,8 @@
           <scan>
             <horizontal>
-              <samples>360</samples>
+              <samples>180</samples> <!--360-->
               <resolution>1</resolution>
-              <min_angle>0.0</min_angle>
-              <max_angle>6.28319</max_angle>
+              <min_angle>-1.5708</min_angle> <!--90:1.5708 0.0 front:0.0rad counterclockwise-->
+              <max_angle>1.5708</max_angle> <!--180:3.14159 270:4.71239 360:6.28319-->
             </horizontal>
           </scan>
